File: hardware/drv8837_breakout/drv8837_breakout.kicad_pcb (KiCad board)
At the start: 2 copper layers, 15.2 x 12.7 mm, 5 parts, among them J1 Conn_01x04_Male, J2 Conn_01x04_Male, U1 DRV8837

Commit message: various updates and drv8837 breakout
Other:
- board text added: "7"
- board text added: "GND"
- board text added: "IN1"
- board text added: "IN2"
- board text added: "OUT1"
- board text added: "OUT2"
- board text added: "SLP"
- board text added: "VCC"
- board text added: "VM"
Changed lines of the file:
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@@
   (general
     (thickness 1.6)
-    (drawings 12)
+    (drawings 22)
     (tracks 34)
     (modules 5)
@@
       (outputformat 1)
       (mirror false)
-      (drillshape 1)
+      (drillshape 0)
       (scaleselection 1)
-      (outputdirectory "")
+      (outputdirectory "plot/")
     )
   )
@@
     (tags "WSON 8 1EP")
     (attr smd)
-    (fp_text reference "U1" (at 0.38 -1.9) (layer "F.SilkS")
+    (fp_text reference "U1" (at 0.902 2.05) (layer "F.SilkS") hide
       (effects (font (size 1 1) (thickness 0.15)))
     )
@@
     )
   )
+  (gr_line (start 153.6 93.2) (end 151 93.2) (layer "B.SilkS") (width 0.12))
+  (gr_text "VCC" (at 153.7 91.3) (layer "B.SilkS")
+    (effects (font (size 1 1) (thickness 0.15)) (justify left mirror))
+  )
+  (gr_text "SLP" (at 153.7 94.1) (layer "B.SilkS")
+    (effects (font (size 1 1) (thickness 0.15)) (justify left mirror))
+  )
+  (gr_text "IN1" (at 153.7 96.6) (layer "B.SilkS")
+    (effects (font (size 1 1) (thickness 0.15)) (justify left mirror))
+  )
+  (gr_text "IN2" (at 153.7 99) (layer "B.SilkS")
+    (effects (font (size 1 1) (thickness 0.15)) (justify left mirror))
+  )
+  (gr_text "GND" (at 145.7 99) (layer "B.SilkS")
+    (effects (font (size 1 1) (thickness 0.15)) (justify right mirror))
+  )
+  (gr_text "OUT2" (at 145.7 96.7) (layer "B.SilkS")
+    (effects (font (size 1 1) (thickness 0.15)) (justify right mirror))
+  )
+  (gr_text "OUT1" (at 145.7 94.1) (layer "B.SilkS")
+    (effects (font (size 1 1) (thickness 0.15)) (justify right mirror))
+  )
+  (gr_text "VM" (at 145.7 91.6) (layer "B.SilkS")
+    (effects (font (size 1 1) (thickness 0.15)) (justify right mirror))
+  )
+  (gr_text "7" (at 152.6 94.5) (layer "F.SilkS")
+    (effects (font (size 1 1) (thickness 0.15)))
+  )
   (gr_text "8" (at 152.4 91.44) (layer "F.SilkS")
