File: hardware/malenki-1616/malenki-1616.kicad_pcb (KiCad board)
At the start: 2 copper layers, 19 x 24.1 mm, 28 parts, among them J1 Conn_01x02_Male, J2 Conn_01x08_Male, J3 Conn_01x02, J5 Conn_01x02_Male, J6 Conn_01x02_Male, J7 Conn_01x02_Male, U1 A7105-MODULE, U2 AIC1734-33GUTR, U3 ATtiny1616-M, U5 DRV8837DSGR, U6 DRV8837DSGR, U7 DRV8837DSGR

Commit message: Capacitor voltage rating
Parts:
- C2, C3, C5, C6, C7: value 10uF -> 10uF 25V
Changed lines of the file:
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@@
     (descr "Capacitor SMD 0603 (1608 Metric), square (rectangular) end terminal, IPC_7351 nominal, (Body size source: IPC-SM-782 page 76, https://www.pcb-3d.com/wordpress/wp-content/uploads/ipc-sm-782a_amendment_1_and_2.pdf), generated with kicad-footprint-generator")
     (tags "capacitor")
-    (property "LCSC" "C19702")
+    (property "LCSC" "C2922482")
     (property "Partnum" "")
     (property "Sheetfile" "malenki-1616.kicad_sch")
@@
       (effects (font (size 1 1) (thickness 0.15)) (justify mirror))
     )
-    (fp_text value "10uF" (at 0 -1.43 180) (layer "B.Fab")
+    (fp_text value "10uF 25V" (at 0 -1.43 180) (layer "B.Fab")
       (effects (font (size 1 1) (thickness 0.15)) (justify mirror))
     )
@@
     (descr "Capacitor SMD 0603 (1608 Metric), square (rectangular) end terminal, IPC_7351 nominal, (Body size source: IPC-SM-782 page 76, https://www.pcb-3d.com/wordpress/wp-content/uploads/ipc-sm-782a_amendment_1_and_2.pdf), generated with kicad-footprint-generator")
     (tags "capacitor")
-    (property "LCSC" "C19702")
+    (property "LCSC" "C2922482")
     (property "Partnum" "")
     (property "Sheetfile" "malenki-1616.kicad_sch")
@@
       (effects (font (size 1 1) (thickness 0.15)) (justify mirror))
     )
-    (fp_text value "10uF" (at 0 -1.43 90) (layer "B.Fab")
+    (fp_text value "10uF 25V" (at 0 -1.43 90) (layer "B.Fab")
       (effects (font (size 1 1) (thickness 0.15)) (justify mirror))
     )
@@
     (descr "Capacitor SMD 0603 (1608 Metric), square (rectangular) end terminal, IPC_7351 nominal, (Body size source: IPC-SM-782 page 76, https://www.pcb-3d.com/wordpress/wp-content/uploads/ipc-sm-782a_amendment_1_and_2.pdf), generated with kicad-footprint-generator")
     (tags "capacitor")
-    (property "LCSC" "C19702")
+    (property "LCSC" "C2922482")
     (property "Partnum" "")
     (property "Sheetfile" "malenki-1616.kicad_sch")
@@
       (effects (font (size 1 1) (thickness 0.15)) (justify mirror))
     )
-    (fp_text value "10uF" (at 0 -1.43) (layer "B.Fab")
+    (fp_text value "10uF 25V" (at 0 -1.43) (layer "B.Fab")
       (effects (font (size 1 1) (thickness 0.15)) (justify mirror))
     )
@@
     (descr "VQFN, 20 Pin (http://ww1.microchip.com/downloads/en/DeviceDoc/20%20Lead%20VQFN%203x3x0_9mm_1_7EP%20U2B%20C04-21496a.pdf), generated with kicad-footprint-generator ipc_noLead_generator.py")
     (tags "VQFN NoLead")
+    (property "LCSC" "C507118")
     (property "Sheetfile" "malenki-1616.kicad_sch")
     (property "Sheetname" "")
@@
     (descr "Capacitor SMD 0603 (1608 Metric), square (rectangular) end terminal, IPC_7351 nominal, (Body size source: IPC-SM-782 page 76, https://www.pcb-3d.com/wordpress/wp-content/uploads/ipc-sm-782a_amendment_1_and_2.pdf), generated with kicad-footprint-generator")
     (tags "capacitor")
-    (property "LCSC" "C19702")
+    (property "LCSC" "C2922482")
     (property "Partnum" "")
     (property "Sheetfile" "malenki-1616.kicad_sch")
@@
       (effects (font (size 1 1) (thickness 0.15)) (justify mirror))
     )
-    (fp_text value "10uF" (at 0 -1.43 90) (layer "B.Fab")
+    (fp_text value "10uF 25V" (at 0 -1.43 90) (layer "B.Fab")
       (effects (font (size 1 1) (thickness 0.15)) (justify mirror))
     )
@@
     (descr "Capacitor SMD 0603 (1608 Metric), square (rectangular) end terminal, IPC_7351 nominal, (Body size source: IPC-SM-782 page 76, https://www.pcb-3d.com/wordpress/wp-content/uploads/ipc-sm-782a_amendment_1_and_2.pdf), generated with kicad-footprint-generator")
     (tags "capacitor")
-    (property "LCSC" "C19702")
+    (property "LCSC" "C2922482")
     (property "Partnum" "")
     (property "Sheetfile" "malenki-1616.kicad_sch")
@@
       (effects (font (size 1 1) (thickness 0.15)) (justify mirror))
     )
-    (fp_text value "10uF" (at 0 -1.43 90) (layer "B.Fab")
-      (effects (font (size 1 1) (thickness 0.15)) (justify mirror))
-    )
+    (fp_text value "10uF 25V" (at 0 -1.43 90) (layer "B.Fab")
+      (effects (font (size 1 1) (thickness 0.15)) (justify mirror))
+    )
