File: hardware/malenki-1616/malenki-1616.kicad_pcb (KiCad board)
At the start: 2 copper layers, 19 x 24.1 mm, 28 parts, among them J1 Conn_01x02_Male, J2 Conn_01x08_Male, J3 Conn_01x02, J5 Conn_01x02_Male, J6 Conn_01x02_Male, J7 Conn_01x02_Male, U1 A7105-MODULE, U2 AIC1734-33GUTR, U3 ATtiny1616-M, U5 DRV8837DSGR, U6 DRV8837DSGR, U7 DRV8837DSGR

Commit message: Malenki 1616 panel update
Parts:
- added REF**: Tab, kikit:Tab, F.Cu at (148.8, 61.6)
- added REF**: Tab, kikit:Tab, F.Cu at (148.8, 86.3)
- added REF**: Tab, kikit:Tab, F.Cu at (155.7, 72.0)
- added REF**: Tab, kikit:Tab, F.Cu at (135.8, 72.0)
Changed lines of the file:
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@@
       (net 39 "unconnected-(J2-Pad8)") (pinfunction "Pin_8") (pintype "passive+no_connect"))
+  )
+  (footprint "kikit:Tab" (layer "F.Cu")
+    (at 148.8 61.6 -90)
+    (descr "A symbol representing annotation for tab placement")
+    (attr exclude_from_pos_files exclude_from_bom)
+    (fp_text reference "REF**" (at 0 -2 90) (layer "F.SilkS") hide
+      (effects (font (size 1 1) (thickness 0.15)))
+    )
+    (fp_text value "Tab" (at -2.75 -1 90) (layer "Dwgs.User")
+      (effects (font (size 1.2 1.2) (thickness 0.2)))
+    )
+    (fp_text user "KIKIT: width: 3mm" (at -5.5 0) (layer "Dwgs.User")
+      (effects (font (size 1 1) (thickness 0.15)))
+    )
+    (fp_line (start 0.25 1) (end 0.25 -1) (layer "Dwgs.User") (width 0.3))
+    (fp_line (start 0.25 0) (end -2.75 0) (layer "Dwgs.User") (width 0.3))
+    (fp_line (start 0.25 0) (end -0.75 -1) (layer "Dwgs.User") (width 0.3))
+    (fp_line (start 0.25 0) (end -0.75 1) (layer "Dwgs.User") (width 0.3))
+  )
+  (footprint "kikit:Tab" (layer "F.Cu")
+    (at 148.8 86.35 90)
+    (descr "A symbol representing annotation for tab placement")
+    (attr exclude_from_pos_files exclude_from_bom)
+    (fp_text reference "REF**" (at 0 -2 90) (layer "F.SilkS") hide
+      (effects (font (size 1 1) (thickness 0.15)))
+    )
+    (fp_text value "Tab" (at -2.75 -1 90) (layer "Dwgs.User")
+      (effects (font (size 1.2 1.2) (thickness 0.2)))
+    )
+    (fp_text user "KIKIT: width: 3mm" (at -5.5 0) (layer "Dwgs.User")
+      (effects (font (size 1 1) (thickness 0.15)))
+    )
+    (fp_line (start 0.25 0) (end -0.75 1) (layer "Dwgs.User") (width 0.3))
+    (fp_line (start 0.25 0) (end -0.75 -1) (layer "Dwgs.User") (width 0.3))
+    (fp_line (start 0.25 1) (end 0.25 -1) (layer "Dwgs.User") (width 0.3))
+    (fp_line (start 0.25 0) (end -2.75 0) (layer "Dwgs.User") (width 0.3))
+  )
+  (footprint "kikit:Tab" (layer "F.Cu")
+    (at 155.7 72 180)
+    (descr "A symbol representing annotation for tab placement")
+    (attr exclude_from_pos_files exclude_from_bom)
+    (fp_text reference "REF**" (at 0 -2) (layer "F.SilkS") hide
+      (effects (font (size 1 1) (thickness 0.15)))
+    )
+    (fp_text value "Tab" (at -2.75 -1) (layer "Dwgs.User")
+      (effects (font (size 1.2 1.2) (thickness 0.2)))
+    )
+    (fp_text user "KIKIT: width: 3mm" (at -5.5 0 90) (layer "Dwgs.User")
+      (effects (font (size 1 1) (thickness 0.15)))
+    )
+    (fp_line (start 0.25 0) (end -0.75 1) (layer "Dwgs.User") (width 0.3))
+    (fp_line (start 0.25 1) (end 0.25 -1) (layer "Dwgs.User") (width 0.3))
+    (fp_line (start 0.25 0) (end -0.75 -1) (layer "Dwgs.User") (width 0.3))
+    (fp_line (start 0.25 0) (end -2.75 0) (layer "Dwgs.User") (width 0.3))
+  )
+  (footprint "kikit:Tab" (layer "F.Cu")
+    (at 135.85 72)
+    (descr "A symbol representing annotation for tab placement")
+    (attr exclude_from_pos_files exclude_from_bom)
+    (fp_text reference "REF**" (at 0 -2) (layer "F.SilkS") hide
+      (effects (font (size 1 1) (thickness 0.15)))
+    )
+    (fp_text value "Tab" (at -2.75 -1) (layer "Dwgs.User")
+      (effects (font (size 1.2 1.2) (thickness 0.2)))
+    )
+    (fp_text user "KIKIT: width: 3mm" (at -5.5 0 90) (layer "Dwgs.User")
+      (effects (font (size 1 1) (thickness 0.15)))
+    )
+    (fp_line (start 0.25 0) (end -2.75 0) (layer "Dwgs.User") (width 0.3))
+    (fp_line (start 0.25 0) (end -0.75 1) (layer "Dwgs.User") (width 0.3))
+    (fp_line (start 0.25 0) (end -0.75 -1) (layer "Dwgs.User") (width 0.3))
+    (fp_line (start 0.25 1) (end 0.25 -1) (layer "Dwgs.User") (width 0.3))
   )
   (footprint "Capacitor_SMD:C_0603_1608Metric" (layer "B.Cu")
@@
   (gr_circle (center 151.4 79.6) (end 151.527 79.6) (layer "B.SilkS") (width 0.5) (fill none))
   (gr_circle (center 143.3 79.6) (end 143.427 79.6) (layer "B.SilkS") (width 0.5) (fill none))
+  (gr_rect (start 136.5 61.4) (end 155.3 61.9) (layer "B.Mask") (width 0.15) (fill solid))
+  (gr_rect (start 136.5 61.4) (end 155.3 61.9) (layer "F.Mask") (width 0.15) (fill solid))
   (gr_line (start 155.4 61.722) (end 136.398 61.722) (layer "Edge.Cuts") (width 0.05))
   (gr_line (start 155.4 84.4) (end 155.4 61.722) (layer "Edge.Cuts") (width 0.05))

Commit message: Malenki 1616 - component swap on voltage reg
Parts:
- U2: value AIC1734-33GUTR -> AP2210N-3.3TRG1
Changed lines of the file:
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@@
     (descr "Capacitor SMD 0603 (1608 Metric), square (rectangular) end terminal, IPC_7351 nominal, (Body size source: IPC-SM-782 page 76, https://www.pcb-3d.com/wordpress/wp-content/uploads/ipc-sm-782a_amendment_1_and_2.pdf), generated with kicad-footprint-generator")
     (tags "capacitor")
-    (property "LCSC" "C2922482")
+    (property "LCSC" "C96446")
     (property "Partnum" "")
     (property "Sheetfile" "malenki-1616.kicad_sch")
@@
     (descr "Capacitor SMD 0603 (1608 Metric), square (rectangular) end terminal, IPC_7351 nominal, (Body size source: IPC-SM-782 page 76, https://www.pcb-3d.com/wordpress/wp-content/uploads/ipc-sm-782a_amendment_1_and_2.pdf), generated with kicad-footprint-generator")
     (tags "capacitor")
-    (property "LCSC" "C2922482")
+    (property "LCSC" "C96446")
     (property "Partnum" "")
     (property "Sheetfile" "malenki-1616.kicad_sch")
@@
     (tags "SOT TO_SOT_SMD")
     (property "LCSC" "C211659")
-    (property "Partnum" "C211659")
+    (property "Partnum" "C155508")
     (property "Sheetfile" "malenki-1616.kicad_sch")
     (property "Sheetname" "")
@@
       (effects (font (size 1 1) (thickness 0.15)) (justify mirror))
     )
-    (fp_text value "AIC1734-33GUTR" (at 0 -2.5 -90) (layer "B.Fab")
+    (fp_text value "AP2210N-3.3TRG1" (at 0 -2.5 -90) (layer "B.Fab")
       (effects (font (size 1 1) (thickness 0.15)) (justify mirror))
     )
@@
     (descr "Capacitor SMD 0603 (1608 Metric), square (rectangular) end terminal, IPC_7351 nominal, (Body size source: IPC-SM-782 page 76, https://www.pcb-3d.com/wordpress/wp-content/uploads/ipc-sm-782a_amendment_1_and_2.pdf), generated with kicad-footprint-generator")
     (tags "capacitor")
-    (property "LCSC" "C2922482")
+    (property "LCSC" "C96446")
     (property "Partnum" "")
     (property "Sheetfile" "malenki-1616.kicad_sch")
@@
     (descr "Capacitor SMD 0603 (1608 Metric), square (rectangular) end terminal, IPC_7351 nominal, (Body size source: IPC-SM-782 page 76, https://www.pcb-3d.com/wordpress/wp-content/uploads/ipc-sm-782a_amendment_1_and_2.pdf), generated with kicad-footprint-generator")
     (tags "capacitor")
-    (property "LCSC" "C2922482")
+    (property "LCSC" "C96446")
     (property "Partnum" "")
     (property "Sheetfile" "malenki-1616.kicad_sch")
@@
     (descr "Capacitor SMD 0603 (1608 Metric), square (rectangular) end terminal, IPC_7351 nominal, (Body size source: IPC-SM-782 page 76, https://www.pcb-3d.com/wordpress/wp-content/uploads/ipc-sm-782a_amendment_1_and_2.pdf), generated with kicad-footprint-generator")
     (tags "capacitor")
-    (property "LCSC" "C2922482")
+    (property "LCSC" "C96446")
     (property "Partnum" "")
     (property "Sheetfile" "malenki-1616.kicad_sch")
