File: hardware/malenki-plus/malenki-plus.kicad_pcb (KiCad board)
At the start: 2 copper layers, 19 x 24.1 mm, 28 parts, among them J1 Conn_01x02_Male, J2 Conn_01x08_Male, J3 Conn_01x02, J5 Conn_01x02_Male, J6 Conn_01x02_Male, J7 Conn_01x02_Male, U1 A7105-MODULE, U2 HT7533-1, U3 ATtiny1616-M, U5 DRV8231DSGR, U6 DRV8231DSGR, U7 DRV8231DSGR

Commit message: Update jlc parts
Parts:
- D1: value LED Blue -> LED White
Changed lines of the file:
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@@
     (descr "Capacitor SMD 0603 (1608 Metric), square (rectangular) end terminal, IPC_7351 nominal, (Body size source: IPC-SM-782 page 76, https://www.pcb-3d.com/wordpress/wp-content/uploads/ipc-sm-782a_amendment_1_and_2.pdf), generated with kicad-footprint-generator")
     (tags "capacitor")
-    (property "LCSC" "C2922482")
+    (property "LCSC" "C96446")
     (property "Partnum" "")
     (property "Sheetfile" "malenki-plus.kicad_sch")
@@
     (descr "Capacitor SMD 0603 (1608 Metric), square (rectangular) end terminal, IPC_7351 nominal, (Body size source: IPC-SM-782 page 76, https://www.pcb-3d.com/wordpress/wp-content/uploads/ipc-sm-782a_amendment_1_and_2.pdf), generated with kicad-footprint-generator")
     (tags "capacitor")
-    (property "LCSC" "C2922482")
+    (property "LCSC" "C96446")
     (property "Partnum" "")
     (property "Sheetfile" "malenki-plus.kicad_sch")
@@
     (descr "LED SMD 0805 (2012 Metric), square (rectangular) end terminal, IPC_7351 nominal, (Body size source: https://docs.google.com/spreadsheets/d/1BsfQQcO9C6DZCsRaXUlFlo91Tg2WpOkGARC1WS5S8t0/edit?usp=sharing), generated with kicad-footprint-generator")
     (tags "LED handsolder")
-    (property "LCSC" "C2293")
+    (property "LCSC" "C34499")
     (property "Sheetfile" "malenki-plus.kicad_sch")
     (property "Sheetname" "")
@@
       (effects (font (size 1 1) (thickness 0.15)) (justify mirror))
     )
-    (fp_text value "LED Blue" (at 0 -1.65 270) (layer "B.Fab")
+    (fp_text value "LED White" (at 0 -1.65 270) (layer "B.Fab")
       (effects (font (size 1 1) (thickness 0.15)) (justify mirror))
     )
@@
     (descr "Capacitor SMD 0603 (1608 Metric), square (rectangular) end terminal, IPC_7351 nominal, (Body size source: IPC-SM-782 page 76, https://www.pcb-3d.com/wordpress/wp-content/uploads/ipc-sm-782a_amendment_1_and_2.pdf), generated with kicad-footprint-generator")
     (tags "capacitor")
-    (property "LCSC" "C2922482")
+    (property "LCSC" "C96446")
     (property "Partnum" "")
     (property "Sheetfile" "malenki-plus.kicad_sch")
@@
     (descr "Capacitor SMD 0603 (1608 Metric), square (rectangular) end terminal, IPC_7351 nominal, (Body size source: IPC-SM-782 page 76, https://www.pcb-3d.com/wordpress/wp-content/uploads/ipc-sm-782a_amendment_1_and_2.pdf), generated with kicad-footprint-generator")
     (tags "capacitor")
-    (property "LCSC" "C2922482")
+    (property "LCSC" "C96446")
     (property "Partnum" "")
     (property "Sheetfile" "malenki-plus.kicad_sch")
@@
     (descr "Capacitor SMD 0603 (1608 Metric), square (rectangular) end terminal, IPC_7351 nominal, (Body size source: IPC-SM-782 page 76, https://www.pcb-3d.com/wordpress/wp-content/uploads/ipc-sm-782a_amendment_1_and_2.pdf), generated with kicad-footprint-generator")
     (tags "capacitor")
-    (property "LCSC" "C2922482")
-    (property "Partnum" "")
-    (property "Sheetfile" "malenki-plus.kicad_sch")
+    (property "LCSC" "C96446")
+    (property "Partnum" "")
+    (property "Sheetfile" "malenki-plus.kicad_sch")
