File: hardware/malenki-plus/malenki-plus.kicad_sch (KiCad schematic)
At the start: 28 parts, among them J1 Conn_01x02_Male, J2 Conn_01x08_Male, J3 Conn_01x02, J5 Conn_01x02_Male, J6 Conn_01x02_Male, J7 Conn_01x02_Male, U1 A7105-MODULE, U2 HT7533-1, U3 ATtiny1616-M, U5 DRV8231DSGR, U6 DRV8231DSGR, U7 DRV8231DSGR

Commit message: Update jlc part numbers
Parts:
- R3: LCSC (none) -> C25741
- R4: LCSC (none) -> C25744
- U2: LCSC (none) -> C14289
Changed lines of the file:
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@@
       (effects (font (size 1.27 1.27)) hide)
     )
-    (property "LCSC" "" (id 5) (at 106.68 152.4 0)
+    (property "LCSC" "C25741" (id 5) (at 106.68 152.4 0)
       (effects (font (size 1.27 1.27)) hide)
     )
@@
       (effects (font (size 1.27 1.27)) hide)
     )
-    (property "LCSC" "" (id 5) (at 106.68 160.02 0)
+    (property "LCSC" "C25744" (id 5) (at 106.68 160.02 0)
       (effects (font (size 1.27 1.27)) hide)
     )
@@
       (effects (font (size 1.27 1.27)) hide)
     )
+    (property "LCSC" "C14289" (id 4) (at 78.74 50.8 0)
+      (effects (font (size 1.27 1.27)) hide)
+    )

Commit message: Update jlc parts
Parts:
- C2, C3, C5, C6, C7: LCSC C2922482 -> C96446
- D1: value LED Blue -> LED White; LCSC C2293 -> C34499
Changed lines of the file:
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@@
       (effects (font (size 1.27 1.27)) hide)
     )
-    (property "LCSC" "C2922482" (id 5) (at 63.5 52.07 0)
+    (property "LCSC" "C96446" (id 5) (at 63.5 52.07 0)
       (effects (font (size 1.27 1.27)) hide)
     )
@@
       (effects (font (size 1.27 1.27)) hide)
     )
-    (property "LCSC" "C2922482" (id 5) (at 92.71 52.07 0)
+    (property "LCSC" "C96446" (id 5) (at 92.71 52.07 0)
       (effects (font (size 1.27 1.27)) hide)
     )
@@
       (effects (font (size 1.27 1.27)) (justify right))
     )
-    (property "Value" "LED Blue" (id 1) (at 133.7818 157.5308 90)
+    (property "Value" "LED White" (id 1) (at 133.7818 157.5308 90)
       (effects (font (size 1.27 1.27)) (justify right))
     )
@@
       (effects (font (size 1.27 1.27)) hide)
     )
-    (property "LCSC" "C2293" (id 4) (at 130.81 156.21 0)
+    (property "LCSC" "C34499" (id 4) (at 130.81 156.21 0)
       (effects (font (size 1.27 1.27)) hide)
     )
@@
       (effects (font (size 1.27 1.27)) hide)
     )
-    (property "LCSC" "C2922482" (id 5) (at 219.71 46.99 0)
+    (property "LCSC" "C96446" (id 5) (at 219.71 46.99 0)
       (effects (font (size 1.27 1.27)) hide)
     )
@@
       (effects (font (size 1.27 1.27)) hide)
     )
-    (property "LCSC" "C2922482" (id 5) (at 217.17 97.79 0)
+    (property "LCSC" "C96446" (id 5) (at 217.17 97.79 0)
       (effects (font (size 1.27 1.27)) hide)
     )
@@
       (effects (font (size 1.27 1.27)) hide)
     )
-    (property "LCSC" "C2922482" (id 5) (at 215.9 147.32 0)
+    (property "LCSC" "C96446" (id 5) (at 215.9 147.32 0)
       (effects (font (size 1.27 1.27)) hide)
     )
@@
     )
     (path "/00000000-0000-0000-0000-00005cdd2ed4"
-      (reference "D1") (unit 1) (value "LED Blue") (footprint "LED_SMD:LED_0805_2012Metric_Pad1.15x1.40mm_HandSolder")
+      (reference "D1") (unit 1) (value "LED White") (footprint "LED_SMD:LED_0805_2012Metric_Pad1.15x1.40mm_HandSolder")
     )
     (path "/00000000-0000-0000-0000-00005d6ab864"
