File: hardware/malenki-nanoi/radio.kicad_sch (KiCad schematic)
At the start: 22 parts, among them U1 A7105, Y1 16mhz Seiko Epson Q24FA20H005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

Commit message: Doc alternative xtal
Other:
- note added: "Alternative Crystal: JGHC S2216000121080 LCSC number C426965"
Changed lines of the file:
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@@
     (effects (font (size 1.27 1.27)) (justify right bottom))
+  )
+  (text "Alternative Crystal:\nJGHC S2216000121080\nLCSC number C426965"
+    (at 162.56 162.56 0)
+    (effects (font (size 1.27 1.27)) (justify left bottom))
   )
   (text "Crystal requirements (from A7105 datasheet)\n- ESR <= 80ohm\nFirmware FC on - accuracy 20ppm\nFirmware FC off - accuracy 10ppm"
