File: hardware/malenki-hv/motor_driver.kicad_sch (KiCad schematic)
At the start: 3 parts, among them J4 Conn_01x02_Male-Connector, U4 DRV8231DSGR

Commit message: Malenki HV update production info
Parts:
- U4: LCSC (none) -> C3681197
Changed lines of the file:
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@@
+      (effects (font (size 1.27 1.27)) hide)
+    )
+    (property "LCSC" "C3681197" (at 147.32 97.79 0)
       (effects (font (size 1.27 1.27)) hide)
     )
