File: hardware/notmalenki/radio.kicad_sch (KiCad schematic)
At the start: 22 parts, among them U1 A7105, Y1 16mhz Seiko Epson Q24FA20H005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

Commit message: Updates for BOM for production
Parts:
- C10: MPN 0402CG220J500NT -> CL31A226KAHNNNE
- C9: MPN 0402CG1R0C500NT -> CL31A226KAHNNNE
- L3: Manufacturer Guangdong Fenghua -> Murata
- R25: Partnum 10k -> (none)
- U1: PartNumber (none) -> A71X05AQFI/Q
- Y1: PartNumber (none) -> Q24FA20H0051200
Changed lines of the file:
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@@
+      (effects (font (size 1.27 1.27)) hide)
+    )
+    (property "PartNumber" "" (at 208.28 140.97 0)
       (effects (font (size 1.27 1.27)) hide)
     )
@@
       (effects (font (size 1.27 1.27)) hide)
     )
+    (property "PartNumber" "" (at 149.86 100.33 0)
+      (effects (font (size 1.27 1.27)) hide)
+    )
     (pin "1")
     (pin "2")
@@
       (effects (font (size 1.27 1.27)) hide)
     )
+    (property "PartNumber" "" (at 128.27 83.82 0)
+      (effects (font (size 1.27 1.27)) hide)
+    )
     (pin "1")
     (pin "2")
@@
       (effects (font (size 1.27 1.27)) hide)
     )
-    (property "MPN" "0402CG220J500NT" (at 128.27 76.2 0)
+    (property "MPN" "CL31A226KAHNNNE" (at 128.27 76.2 0)
       (effects (font (size 1.27 1.27)) hide)
     )
@@
       (effects (font (size 1.27 1.27)) hide)
     )
+    (property "PartNumber" "" (at 128.27 76.2 0)
+      (effects (font (size 1.27 1.27)) hide)
+    )
     (pin "1")
     (pin "2")
@@
       (effects (font (size 1.27 1.27)) hide)
     )
+    (property "PartNumber" "" (at 228.6 140.97 0)
+      (effects (font (size 1.27 1.27)) hide)
+    )
     (pin "1")
     (pin "2")
@@
     )
     (property "Manufacturer" "AMICCOM" (at 217.17 76.2 0)
+      (effects (font (size 1.27 1.27)) hide)
+    )
+    (property "PartNumber" "A71X05AQFI/Q" (at 217.17 76.2 0)
       (effects (font (size 1.27 1.27)) hide)
     )
@@
       (effects (font (size 1.27 1.27)) hide)
     )
+    (property "PartNumber" "" (at 223.52 112.395 0)
+      (effects (font (size 1.27 1.27)) hide)
+    )
     (pin "1")
     (pin "2")
@@
       (effects (font (size 1.27 1.27)) hide)
     )
+    (property "PartNumber" "" (at 113.03 94.615 0)
+      (effects (font (size 1.27 1.27)) hide)
+    )
     (pin "1")
     (pin "2")
@@
       (effects (font (size 1.27 1.27)) hide)
     )
-    (property "Partnum" "10k" (at 199.39 109.22 0)
+    (property "PartNumber" "" (at 199.39 109.22 0)
       (effects (font (size 1.27 1.27)) hide)
     )
@@
       (effects (font (size 1.27 1.27)) hide)
     )
+    (property "PartNumber" "" (at 189.23 109.22 0)
+      (effects (font (size 1.27 1.27)) hide)
+    )
     (pin "1")
     (pin "2")
@@
       (effects (font (size 1.27 1.27)) hide)
     )
+    (property "PartNumber" "" (at 196.85 59.69 0)
+      (effects (font (size 1.27 1.27)) hide)
+    )
     (pin "1")
     (pin "2")
@@
       (effects (font (size 1.27 1.27)) hide)
     )
-    (property "MPN" "0402CG1R0C500NT" (at 99.06 80.01 0)
+    (property "MPN" "CL31A226KAHNNNE" (at 99.06 80.01 0)
       (effects (font (size 1.27 1.27)) hide)
     )
@@
       (effects (font (size 1.27 1.27)) hide)
     )
+    (property "PartNumber" "" (at 99.06 80.01 0)
+      (effects (font (size 1.27 1.27)) hide)
+    )
     (pin "1")
     (pin "2")
@@
     )
     (property "Manufacturer" "Samsung" (at 203.2 45.72 0)
+      (effects (font (size 1.27 1.27)) hide)
+    )
+    (property "PartNumber" "" (at 203.2 45.72 0)
       (effects (font (size 1.27 1.27)) hide)
     )
@@
       (effects (font (size 1.27 1.27)) hide)
     )
+    (property "PartNumber" "" (at 59.69 73.66 0)
+      (effects (font (size 1.27 1.27)) hide)
+    )
     (pin "1")
     (pin "2")
@@
     )
     (property "Manufacturer" "Seiko Epson" (at 218.44 137.16 0)
+      (effects (font (size 1.27 1.27)) hide)
+    )
+    (property "PartNumber" "Q24FA20H0051200" (at 218.44 137.16 0)
       (effects (font (size 1.27 1.27)) hide)
     )
@@
       (effects (font (size 1.27 1.27)) hide)
     )
-    (property "Manufacturer" "Guangdong Fenghua" (at 149.86 82.55 0)
+    (property "Manufacturer" "Murata" (at 149.86 82.55 0)
+      (effects (font (size 1.27 1.27)) hide)
+    )
+    (property "PartNumber" "" (at 149.86 82.55 0)
       (effects (font (size 1.27 1.27)) hide)
     )
@@
       (effects (font (size 1.27 1.27)) hide)
     )
+    (property "PartNumber" "" (at 144.78 64.77 0)
+      (effects (font (size 1.27 1.27)) hide)
+    )
     (pin "1")
     (pin "2")
@@
       (effects (font (size 1.27 1.27)) hide)
     )
+    (property "PartNumber" "" (at 91.44 76.2 0)
+      (effects (font (size 1.27 1.27)) hide)
+    )
     (pin "1")
     (pin "2")
@@
       (effects (font (size 1.27 1.27)) hide)
     )
+    (property "PartNumber" "" (at 189.23 100.33 0)
+      (effects (font (size 1.27 1.27)) hide)
+    )
     (pin "1")
     (pin "2")
@@
       (effects (font (size 1.27 1.27)) hide)
     )
+    (property "PartNumber" "" (at 177.8 64.77 0)
+      (effects (font (size 1.27 1.27)) hide)
+    )
     (pin "1")
     (pin "2")
@@
       (effects (font (size 1.27 1.27)) hide)
     )
+    (property "PartNumber" "" (at 162.56 88.9 0)
+      (effects (font (size 1.27 1.27)) hide)
+    )
     (pin "1")
     (pin "2")
@@
       (effects (font (size 1.27 1.27)) hide)
     )
+    (property "PartNumber" "" (at 243.84 83.82 0)
+      (effects (font (size 1.27 1.27)) hide)
+    )

Commit message: Schematic notes
Parts:
- Y1: value 16mhz Seiko Epson Q24FA20H0051200 -> 16mhz Seiko Epson Q24FA20H00512; MPN Q24FA20H0051200 -> Q24FA20H00512; PartNumber Q24FA20H0051200 -> Q24FA20H00512
Changed lines of the file:
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@@
       (effects (font (size 1.27 1.27)) (justify left))
     )
-    (property "Value" "16mhz Seiko Epson Q24FA20H0051200 " (at 213.36 128.27 0)
+    (property "Value" "16mhz Seiko Epson Q24FA20H00512" (at 213.36 128.27 0)
       (effects (font (size 1.27 1.27)) (justify left))
     )
@@
       (effects (font (size 1.27 1.27)) hide)
     )
-    (property "MPN" "Q24FA20H0051200" (at 218.44 137.16 0)
+    (property "MPN" "Q24FA20H00512" (at 218.44 137.16 0)
       (effects (font (size 1.27 1.27)) hide)
     )
@@
       (effects (font (size 1.27 1.27)) hide)
     )
-    (property "PartNumber" "Q24FA20H0051200" (at 218.44 137.16 0)
+    (property "PartNumber" "Q24FA20H00512" (at 218.44 137.16 0)
       (effects (font (size 1.27 1.27)) hide)
     )
